File: cad/kicad/controller/ind-sense.sch (KiCad schematic (older format))
At the start: 22 parts, among them J1 Conn_01x27, J2 Conn_01x27, J3 Conn_01x18, U1 74HC154, U2 MCP4821, U5 CMP04, U6 CMP04

Commit message: seperated the controller from the demo macropad, remade the controller to hopefully be less succeptable to emi, and digital interferance.
Parts:
- removed J2: Conn_01x27, Pin_Headers:Pin_Header_Straight_1x27_Pitch2.54mm, symbol Conn_01x27
- C1: renamed from C9; value 1u -> 0u1
- C2: footprint Capacitors_SMD:C_0805_HandSoldering -> Capacitors_SMD:C_0603_HandSoldering
- C5: renamed from C4; value 1u -> 0u1
- C7: renamed from C5; value 1u -> 0u1
- renumbered C1 to C3, C3 to C4, C13 to C6, C18 to C8, J3 to J2, R4 to R1, R5 to R2, R6 to R3, U5 to U3, U6 to U4
Connections:
- net M1: now also U3.8 (-); no longer U3.10 (-)
- net M2: now also U3.10 (-); no longer U3.8 (-)
- net M5: now also U4.8 (-); no longer U4.10 (-)
- net M6: now also U4.10 (-); no longer U4.8 (-)
- net S1: now also RN3.4 (R4.1), U3.14; no longer RN3.3 (R3.1), U3.13
- net S2: now also RN3.3 (R3.1), U3.13; no longer RN3.4 (R4.1), U3.14
- net S5: now also RN4.4 (R4.1), U4.14; no longer RN4.3 (R3.1), U4.13
- net S6: now also RN4.3 (R3.1), U4.13; no longer RN4.4 (R4.1), U4.14
- net SDI: now also J2.2 (Pin_2); no longer J2.4 (Pin_4)
- net ~SS: now also J2.4 (Pin_4); no longer J2.2 (Pin_2)
Other:
- moved on the sheet: C1, C3, C4, R1, R2, R3, U1, U2

Commit message: updated controller with a lower part count equivalent, that should also be more accurate. need to have an actuall EE review the board and it's design
Parts:
- removed J2: Conn_01x18, Pin_Headers:Pin_Header_Straight_1x18_Pitch2.54mm, symbol Conn_01x18
- removed RN3, RN4: 66k, Resistors_SMD:R_Array_Convex_4x0402, symbol R_Pack04
- removed U3, U4: CMP04, Housings_SSOP:TSSOP-14_4.4x5mm_Pitch0.65mm, symbol LM339
- added C10, C9: 0u1, Capacitors_SMD:C_0603_HandSoldering, symbol C_Small
- added D1, D2, D3, D4: ~, Diodes_SMD:D_0603, symbol D_Schottky_Small_ALT
- added J2: Conn_01x16, Pin_Headers:Pin_Header_Straight_1x16_Pitch2.54mm, symbol Conn_01x16
- added U3: NX3L4051, Housings_SSOP:TSSOP-16_4.4x5mm_Pitch0.65mm, symbol NX3L4051
- added U4: LMV761, TO_SOT_Packages_SMD:SOT-23-6_Handsoldering, symbol LMV761
- C2: value 100u -> 0u1
- RN1, RN2: value 330 -> 2k64
Connections:
- net +3V3: now also C5.1, C10.2, D3.2 (A), D4.1 (K), U3.16 (VDD); no longer C2.1, C3.1, C4.1, C6.1, C8.1, R2.1, U2.1 (Vdd)
- net GND: now also C8.1, D1.2 (A), D2.1 (K), U3.8 (VSS), U4.5 (~SD); no longer C3.2, C4.2, C6.2, C7.2, C8.2, J1.1 (Pin_1), J1.11 (Pin_11), J1.12 (Pin_12), J1.2 (Pin_2), J1.26 (Pin_26), J1.27 (Pin_27), R3.2, U2.7 (Vss)
- net M1: now also RN1.5 (R4.2), U3.5 (X5); no longer RN1.4 (R4.1)
- net M2: now also RN1.6 (R3.2), U3.4 (X7); no longer RN1.3 (R3.1)
- net M3: now also RN1.7 (R2.2), U3.2 (X6); no longer RN1.2 (R2.1)
- net M4: now also RN1.8 (R1.2), U3.1 (X4); no longer RN1.1 (R1.1)
- net M5: now also RN2.1 (R1.1), U3.15 (X2); no longer RN2.4 (R4.1)
- net M6: now also RN2.2 (R2.1), U3.14 (X1); no longer RN2.3 (R3.1)
- net M7: now also RN2.3 (R3.1), U3.13 (X0); no longer RN2.2 (R2.1)
- net M8: now also RN2.4 (R4.1), U3.12 (X3); no longer RN2.1 (R1.1)
- net SCK: now also J2.3 (Pin_3)
- net SDI: now also J2.2 (Pin_2)
- net ~SS: now also J2.4 (Pin_4)
- net SEL1 renamed CSEL1
- net CSEL1: now also J2.10 (Pin_10)
- net SEL2 renamed CSEL2
- net CSEL2: now also J2.11 (Pin_11)
- net SEL3 renamed CSEL3
- net CSEL3: now also J2.12 (Pin_12)
- net SEL4 renamed CSEL4
- net CSEL4: now also J2.13 (Pin_13)
- net SP: no longer names the net of R1.2, R2.2, R3.1
- net SP: now also C6.1, U4.3 (-); no longer C5.1, C7.1
- net ~STROBE renamed ~CSTROBE
- net ~CSTROBE: now also J2.14 (Pin_14)
- new net: U3.3 (X), U4.1 (+)
- new net +3.3VA: C3.1, C4.1, C7.1, C9.2, D3.1 (K), D4.2 (A), R2.1, RN1.1 (R1.1), RN1.2 (R2.1), RN1.3 (R3.1), RN1.4 (R4.1), RN2.5 (R4.2), RN2.6 (R3.2), RN2.7 (R2.2), RN2.8 (R1.2), U2.1 (Vdd), U4.6 (V+)
- new net +3.3VP: C10.1, C9.1, J2.1 (Pin_1)
- new net GNDA: C2.1, C3.2, C4.2, C6.2, C7.2, D1.1 (K), D2.2 (A), R3.2, U2.7 (Vss), U4.2 (V-)
- new net GNDREF: C2.2, C8.2, J1.1 (Pin_1), J1.11 (Pin_11), J1.12 (Pin_12), J1.2 (Pin_2), J1.26 (Pin_26), J1.27 (Pin_27), J2.16 (Pin_16)
- new net OUT: J2.5 (Pin_5), U4.4
- new net RSEL1: J2.7 (Pin_7), U3.11 (A)
- new net RSEL2: J2.8 (Pin_8), U3.10 (B)
- new net RSEL3: J2.9 (Pin_9), U3.9 (C)
- new net ~RSTROBE: J2.6 (Pin_6), U3.6 (Inh)
- no-connect marks 3 -> 4
Other:
- moved on the sheet: C4, R1, R2, R3, U2
